File: electronics/main controller/tmc2209.sch (EAGLE design)
At the start: 6 parts, among them J1 JST-PH3

Commit message: pre-production PCBs
Parts:
- removed D1: (no value), adafruit:DIODESOD-123
- removed J1: JST-PH3, jst-ph:JST-PH3
- removed Q1: (no value), adafruit:MOSFET-NREFLOW
- added AUX-X, AUX-Y, AUX-Z, DRV-X, DRV-Y, DRV-Z: (no value), SparkFun-Connectors:M06LOCK
- added C10, C14, C15, C16, C17, C2, C21, C3, C7, C8, C9: 100n, adafruit:C-USC0603
- added C11, C18, C4: 2.2u, adafruit:C-USC1206
- added C12, C19, C5: 22n, adafruit:C-USC0603
- added C13, C20, C6: 10u, adafruit:C-USC1206
- added PDX, PDY, PDZ, SJ10, SJ11, SJ12, SJ2, SJ3, SJ5, SJ6, SJ8, SJ9: SOLDERJUMPERNO, SparkFun-Retired:SOLDERJUMPERNO
- added R10, R5, R6, R9: (no value), adafruit:R-US_R0805
- added R11, R12, R3, R4, R7, R8: (no value), adafruit:R-US_R0603
- added STANDOFF1, STANDOFF2, STANDOFF3, STANDOFF4: STAND-OFFTIGHT, SparkFun-Electromechanical:STAND-OFFTIGHT
- added STEPPER-X, STEPPER-Y, STEPPER-Z: JST-PH5, jst-ph:JST-PH5
- added U1, U2, U3: TMC2209-LA, borkedlabs-powerics:TMC2209-LA
- C1: device adafruit:C-USC1206 -> adafruit:C-USC0603
- R1: value 330 -> (none); device adafruit:R-US_R1206 -> adafruit:R-US_R0805
- R2: value 10k -> (none); device adafruit:R-US_R1206 -> adafruit:R-US_R0805
Connections:
- removed net GATE: Q1.G, R1.2, R2.2
- removed net M1: C1.1, D1.C, J1.1
- removed net M2: C1.2, D1.A, Q1.D
- new net 12VX: C15.1, C16.1, C17.2, C20.1, DRV-X.1, U3.VS@22, U3.VS@28
- new net 12VY: C10.2, C13.1, C8.1, C9.1, DRV-Y.1, U2.VS@22, U2.VS@28
- new net 12VZ: C1.1, C2.1, C3.2, C6.1, DRV-Z.1, U1.VS@22, U1.VS@28
- new net 5VX: C21.1, DRV-X.3, R11.1, SJ12.1, SJ8.1, SJ9.1, U3.VCC_IO
- new net 5VY: C14.1, DRV-Y.3, R7.1, SJ11.1, SJ5.1, SJ6.1, U2.VCC_IO
- new net 5VZ: C7.1, DRV-Z.3, R3.1, SJ10.1, SJ2.1, SJ3.1, U1.VCC_IO
- new net DIAGX: AUX-X.3, U3.DIAG
- new net DIAGY: AUX-Y.3, U2.DIAG
- new net DIAGZ: AUX-Z.3, U1.DIAG
- new net DIRX: DRV-X.5, U3.DIR
- new net DIRY: DRV-Y.5, U2.DIR
- new net DIRZ: DRV-Z.5, U1.DIR
- new net ENX: DRV-X.6, U3.ENN
- new net ENY: DRV-Y.6, U2.ENN
- new net ENZ: DRV-Z.6, U1.ENN
- new net INDEXX: AUX-X.2, U3.INDEX
- new net INDEXY: AUX-Y.2, U2.INDEX
- new net INDEXZ: AUX-Z.2, U1.INDEX
- new net N$1: STEPPER-Z.5, U1.OB2
- new net N$10: STEPPER-X.3, U3.OA1
- new net N$11: STEPPER-X.4, U3.OB1
- new net N$12: STEPPER-X.5, U3.OB2
- new net N$13: R5.1, U2.BRA
- new net N$14: C11.1, U2.5VOUT
- new net N$15: SJ2.2, U1.MS1_ADO
- new net N$16: SJ3.2, U1.MS2_AD2
- new net N$17: SJ6.2, U2.MS2_AD2
- new net N$18: R6.1, U2.BRB
- new net N$19: C18.1, U3.5VOUT
- new net N$2: STEPPER-Z.4, U1.OB1
- new net N$20: C17.1, U3.VCP
- new net N$22: C12.2, U2.CPI
- new net N$23: C12.1, U2.CPO
- new net N$24: C19.2, U3.CPI
- new net N$25: SJ5.2, U2.MS1_ADO
- new net N$26: C19.1, U3.CPO
- new net N$27: SJ12.2, U3.SPREAD
- new net N$28: SJ11.2, U2.SPREAD
- new net N$29: SJ9.2, U3.MS2_AD2
- new net N$30: SJ8.2, U3.MS1_ADO
- new net N$31: R11.2, R12.2, U3.VREF
- new net N$32: R7.2, R8.2, U2.VREF
- new net N$34: C10.1, U2.VCP
- new net N$4: STEPPER-Z.2, U1.OA2
- new net N$40: SJ10.2, U1.SPREAD
- new net N$5: STEPPER-Y.5, U2.OB2
- new net N$51: R9.1, U3.BRA
- new net N$52: R10.1, U3.BRB
- new net N$53: R1.1, U1.BRA
- new net N$54: R2.1, U1.BRB
- new net N$55: R3.2, R4.2, U1.VREF
- new net N$56: C4.1, U1.5VOUT
- new net N$57: C5.2, U1.CPI
- new net N$58: C5.1, U1.CPO
- new net N$59: C3.1, U1.VCP
- new net N$6: STEPPER-Y.4, U2.OB1
- new net N$7: STEPPER-Y.3, U2.OA1
- new net N$8: STEPPER-Y.2, U2.OA2
- new net N$9: STEPPER-X.2, U3.OA2
- new net STEPX: DRV-X.4, U3.STEP
- new net STEPY: DRV-Y.4, U2.STEP
- new net STEPZ: DRV-Z.4, U1.STEP
- new net UARTX: AUX-X.1, PDX.2, U3.PDN_UART
- new net UARTY: AUX-Y.1, PDY.2, U2.PDN_UART
- new net UARTZ: AUX-Z.1, PDZ.2, U1.PDN_UART
- net GND: now also C1.2, C11.2, C13.2, C14.2, C15.2, C16.2, C18.2, C2.2, C20.2, C21.2, C4.2, C6.2, C7.2, C8.2, C9.2, DRV-X.2, DRV-Y.2, DRV-Z.2, PDX.1, PDY.1, PDZ.1, R1.2, R10.2, R12.1, R2.2, R4.1, R5.2, R6.2, R8.1, R9.2, U1.CLK, U1.GND@18, U1.GND@3, U1.PAD, U1.STDBY, U2.CLK, U2.GND@18, U2.GND@3, U2.PAD, U2.STDBY, U3.CLK, U3.GND@18, U3.GND@3, U3.PAD, U3.STDBY; no longer J1.3, Q1.S, R2.1
- net N$3: now also STEPPER-Z.3, U1.OA1; no longer J1.2, R1.1
Other:
- moved on the sheet: C1, R1, R2
