File: electronics/main controller/baseboard.sch (EAGLE design)
At the start: 45 parts, among them J1 2.1MMJACKTHM, J2 M02PTH, U1 ATMEGA328P, X1 16MHz

Commit message: updated all PCBs and added PDF schematics
Parts:
- added U$1, U$2: FIDUCIAL, adafruit:FIDUCIAL
Changed lines of the file:
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@@
 <part name="GND6" library="SparkFun-Aesthetics" deviceset="GND" device=""/>
 <part name="GND7" library="SparkFun-Aesthetics" deviceset="GND" device=""/>
+<part name="U$1" library="adafruit" deviceset="FIDUCIAL" device=""/>
+<part name="U$2" library="adafruit" deviceset="FIDUCIAL" device=""/>
 </parts>
 <sheets>
@@
 <instance part="GND6" gate="1" x="246.38" y="33.02"/>
 <instance part="GND7" gate="1" x="254" y="55.88"/>
+<instance part="U$1" gate="G$1" x="116.84" y="121.92"/>
+<instance part="U$2" gate="G$1" x="124.46" y="121.92"/>
 </instances>
 <busses>
