File: electronics/head mounted controller/m328p.brd (EAGLE design)
At the start: 60 x 30 mm, 40 parts, among them J2 M02PTH, U1 ATMEGA328P, U2 V_REG_MIC2920, X1 16MHz

Commit message: pre-production PCBs
Parts:
- removed U$1, U$2: JST-PH3, jst-ph:JST-PH3
- added HEAD-DATA, HEAD-PWR: (no value), jst-ph:JST-PH2
- LIM-X, LIM-Y, LIM-Z: value JST-PH3 -> (none); device jst-ph:JST-PH3 -> jst-ph:JST-PH2
- moved D1 7.02 mm to (15.0, 24.0), turned to 90 degrees
- moved R1 7.00 mm to (15.0, 21.0), turned to 180 degrees
- moved C10 1.00 mm to (15.0, 18.0)
- moved C11 1.00 mm to (15.0, 15.0)
- moved C8 1.00 mm to (9.00, 18.0)
- moved C9 1.00 mm to (9.00, 15.0)
- moved LIM-X 0.50 mm to (56.5, 11.0)
- moved LIM-Y 0.50 mm to (56.5, 16.5)
- moved LIM-Z 0.50 mm to (56.5, 22.0)
- moved U2 0.50 mm to (11.5, 10.0)
Connections:
- net 12V: now also HEAD-PWR.1; no longer U$1.1
- net GND: now also HEAD-PWR.2, U2.4; no longer U$1.2
- net RX: now also HEAD-DATA.1; no longer U$2.1
- net TX: now also HEAD-DATA.2; no longer U$2.2
Routing:
- net LIMY: track 32.4 -> 35.4 mm
- net LIMX: track 31.4 -> 34.4 mm
- net LIMZ: track 38.8 -> 41.8 mm
- net 12V: track 76.8 -> 78.9 mm
Other:
- board text added: "HEAD DATA"
- board text added: "HEAD PWR"

Commit message: updated all PCBs and added PDF schematics
Parts:
- added U$1, U$2: FIDUCIAL, adafruit:FIDUCIAL_1MM
- moved C12 2.00 mm to (13.0, 5.00)
Routing:
- net 5V: track 32.9 -> 34.9 mm
