File: electronics/stepper driver/tmc2209.brd (EAGLE design)
At the start: 60 x 30 mm, 61 parts, among them U1 TMC2209-LA, U2 TMC2209-LA, U3 TMC2209-LA

Commit message: updated all PCBs and added PDF schematics
Parts:
- added U$1, U$2: FIDUCIAL, adafruit:FIDUCIAL_1MM
