File: electronics/vacuum pump board/pump-board.brd (EAGLE design)
At the start: 24 x 24 mm, 5 parts, among them J1 JST-PH3

Commit message: pre-production PCBs
Parts:
- added C1: 100n, adafruit:C1206
- R1, R2: device adafruit:R0805 -> adafruit:R1206
- moved Q1 1.50 mm to (16.5, 10.0)
- moved R2 1.50 mm to (13.5, 10.0)
- moved R1 1.00 mm to (11.0, 10.0)
- moved D1 0.50 mm to (8.50, 10.0)
Connections:
- net M1: now also C1.1
- net M2: now also C1.2
Routing:
- net GND: track 0.00 -> 2.70 mm
- net GATE: track 5.53 -> 6.91 mm
- net N$3: track 5.83 -> 4.99 mm
- net M1: track 12.3 -> 13.1 mm
Changed lines of the file:
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@@
 <layer number="43" name="vRestrict" color="2" fill="10" visible="no" active="yes"/>
 <layer number="44" name="Drills" color="7" fill="1" visible="no" active="yes"/>
-<layer number="45" name="Holes" color="7" fill="1" visible="yes" active="yes"/>
-<layer number="46" name="Milling" color="3" fill="1" visible="yes" active="yes"/>
+<layer number="45" name="Holes" color="7" fill="1" visible="no" active="yes"/>
+<layer number="46" name="Milling" color="3" fill="1" visible="no" active="yes"/>
 <layer number="47" name="Measures" color="7" fill="1" visible="no" active="yes"/>
 <layer number="48" name="Document" color="7" fill="1" visible="no" active="yes"/>
@@
 </autorouter>
 <elements>
-<element name="Q1" library="adafruit" package="SOT23" value="" x="15" y="10" smashed="yes">
-<attribute name="NAME" x="14.345" y="12.655" size="0.8" layer="25"/>
-<attribute name="VALUE" x="13.095" y="6.825" size="1.27" layer="27"/>
-</element>
-<element name="R1" library="adafruit" package="R0805" value="330" x="10" y="10" smashed="yes" rot="R90">
-<attribute name="NAME" x="9.488" y="12.766" size="0.8" layer="25"/>
-<attribute name="VALUE" x="12.286" y="9.238" size="1.27" layer="27" rot="R90"/>
-</element>
-<element name="D1" library="adafruit" package="SOD-123" value="" x="8" y="10" smashed="yes" rot="R90">
-<attribute name="NAME" x="7.4" y="12.75" size="0.8" layer="25"/>
-<attribute name="VALUE" x="9.284" y="8.9" size="0.4064" layer="27" rot="R90"/>
+<element name="Q1" library="adafruit" package="SOT23" value="" x="16.5" y="10" smashed="yes">
+<attribute name="NAME" x="15.845" y="12.655" size="0.8" layer="25"/>
+<attribute name="VALUE" x="14.595" y="6.825" size="1.27" layer="27"/>
+</element>
+<element name="R1" library="adafruit" package="R1206" value="330" x="11" y="10" smashed="yes" rot="R90">
+<attribute name="NAME" x="10.488" y="12.766" size="0.8" layer="25"/>
+<attribute name="VALUE" x="13.286" y="9.238" size="1.27" layer="27" rot="R90"/>
+</element>
+<element name="D1" library="adafruit" package="SOD-123" value="" x="8.5" y="10" smashed="yes" rot="R90">
+<attribute name="NAME" x="7.9" y="12.75" size="0.8" layer="25"/>
+<attribute name="VALUE" x="9.784" y="8.9" size="0.4064" layer="27" rot="R90"/>
 </element>
 <element name="J1" library="jst-ph" package="JST-PH3" value="JST-PH3" x="12" y="4" smashed="yes" rot="R180"/>
-<element name="R2" library="adafruit" package="R0805" value="10k" x="12" y="10" smashed="yes" rot="R90">
-<attribute name="NAME" x="11.488" y="12.766" size="0.8" layer="25"/>
-<attribute name="VALUE" x="14.286" y="9.238" size="1.27" layer="27" rot="R90"/>
+<element name="R2" library="adafruit" package="R1206" value="10k" x="13.5" y="10" smashed="yes" rot="R90">
+<attribute name="NAME" x="12.988" y="12.766" size="0.8" layer="25"/>
+<attribute name="VALUE" x="15.786" y="9.238" size="1.27" layer="27" rot="R90"/>
+</element>
+<element name="C1" library="adafruit" package="C1206" value="100n" x="6" y="10" smashed="yes" rot="R90">
+<attribute name="NAME" x="5.111" y="12.766" size="0.8" layer="25"/>
+<attribute name="VALUE" x="8.286" y="9.111" size="1.27" layer="27" rot="R90"/>
 </element>
 </elements>
@@
 <contactref element="R1" pad="2"/>
 <contactref element="R2" pad="2"/>
-<wire x1="10" y1="11" x2="12" y2="11" width="0.25" layer="1"/>
-<wire x1="14.05" y1="8.9" x2="14.05" y2="9.95" width="0.25" layer="1"/>
-<wire x1="14.05" y1="9.95" x2="13" y2="11" width="0.25" layer="1"/>
-<wire x1="13" y1="11" x2="12" y2="11" width="0.25" layer="1"/>
+<wire x1="11" y1="11.422" x2="13.5" y2="11.422" width="0.25" layer="1"/>
+<wire x1="14.75" y1="11.25" x2="14.75" y2="9" width="0.25" layer="1"/>
+<wire x1="14.75" y1="9" x2="14.85" y2="8.9" width="0.25" layer="1"/>
+<wire x1="14.85" y1="8.9" x2="15.55" y2="8.9" width="0.25" layer="1"/>
+<wire x1="14.75" y1="11.25" x2="14.578" y2="11.422" width="0.25" layer="1"/>
+<wire x1="14.578" y1="11.422" x2="13.5" y2="11.422" width="0.25" layer="1"/>
 </signal>
 <signal name="M2">
@@
 <vertex x="24" y="0"/>
 </polygon>
+<contactref element="C1" pad="2"/>
 </signal>
 <signal name="GND">
@@
 </polygon>
 <polygon width="0.25" layer="1" isolate="0.5" thermals="no" rank="5">
-<vertex x="0" y="8.5"/>
-<vertex x="15.5" y="8.5"/>
-<vertex x="15.5" y="9.5"/>
+<vertex x="0" y="7"/>
+<vertex x="17" y="7"/>
+<vertex x="17" y="9.5"/>
 <vertex x="24" y="9.5"/>
 <vertex x="24" y="0"/>
 <vertex x="0" y="0"/>
 </polygon>
+<wire x1="13.5" y1="8.578" x2="13" y2="8" width="0.5" layer="1"/>
+<wire x1="13.5" y1="8.578" x2="13.5" y2="7" width="0.5" layer="1"/>
+<wire x1="13.5" y1="7" x2="13.75" y2="6.75" width="0.5" layer="1"/>
 </signal>
 <signal name="N$3">
 <contactref element="J1" pad="2"/>
 <contactref element="R1" pad="1"/>
-<wire x1="10" y1="9" x2="10" y2="6" width="0.25" layer="1"/>
-<wire x1="10" y1="6" x2="12" y2="4" width="0.25" layer="1"/>
+<wire x1="11" y1="8.578" x2="11" y2="5" width="0.25" layer="1"/>
+<wire x1="11" y1="5" x2="12" y2="4" width="0.25" layer="1"/>
 </signal>
 <signal name="M1">
@@
 <vertex x="3" y="14"/>
 </polygon>
-<wire x1="10" y1="4" x2="8" y2="6" width="0.5" layer="1"/>
-<wire x1="8" y1="8.15" x2="2.85" y2="8.15" width="0.5" layer="1"/>
+<wire x1="10" y1="4" x2="8.5" y2="5.5" width="0.5" layer="1"/>
 <wire x1="2.85" y1="8.15" x2="2" y2="9" width="0.5" layer="1"/>
 <wire x1="2" y1="9" x2="2" y2="10" width="0.5" layer="1"/>
-<wire x1="8" y1="6" x2="8" y2="8.15" width="0.5" layer="1"/>
+<wire x1="8.5" y1="5.5" x2="8.5" y2="8.15" width="0.5" layer="1"/>
+<contactref element="C1" pad="1"/>
+<wire x1="2.85" y1="8.15" x2="6" y2="8.15" width="0.5" layer="1"/>
+<wire x1="6" y1="8.15" x2="6" y2="8.6" width="0.5" layer="1"/>
+<wire x1="6" y1="8.15" x2="8.5" y2="8.15" width="0.5" layer="1"/>
 </signal>
 </signals>
+<errors>
+</errors>
 </board>
 </drawing>

Commit message: updated all PCBs and added PDF schematics
Parts:
- added U$1, U$2: FIDUCIAL, adafruit:FIDUCIAL_1MM
Changed lines of the file:
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@@
 <wire x1="21.5" y1="13" x2="22" y2="13.5" width="0.001" layer="46" curve="-90"/>
 <wire x1="22" y1="13.5" x2="22.5" y2="13" width="0.001" layer="46" curve="-90"/>
-<text x="8" y="6" size="0.8" layer="25" ratio="10">12V</text>
-<text x="11" y="6" size="0.8" layer="25" ratio="10">SIG</text>
-<text x="13.5" y="6" size="0.8" layer="25" ratio="10">GND</text>
+<text x="8" y="6" size="0.8" layer="25" font="vector" ratio="10">12V</text>
+<text x="11" y="6" size="0.8" layer="25" font="vector" ratio="10">SIG</text>
+<text x="13.5" y="6" size="0.8" layer="25" font="vector" ratio="10">GND</text>
 </plain>
 <attributes>
@@
 <elements>
 <element name="Q1" library="adafruit" package="SOT23" value="" x="16.5" y="10" smashed="yes">
-<attribute name="NAME" x="15.845" y="12.655" size="0.8" layer="25"/>
+<attribute name="NAME" x="15.845" y="12.655" size="0.8" layer="25" font="vector"/>
 <attribute name="VALUE" x="14.595" y="6.825" size="1.27" layer="27"/>
 </element>
 <element name="R1" library="adafruit" package="R1206" value="330" x="11" y="10" smashed="yes" rot="R90">
-<attribute name="NAME" x="10.488" y="12.766" size="0.8" layer="25"/>
+<attribute name="NAME" x="10.488" y="12.766" size="0.8" layer="25" font="vector"/>
 <attribute name="VALUE" x="13.286" y="9.238" size="1.27" layer="27" rot="R90"/>
 </element>
 <element name="D1" library="adafruit" package="SOD-123" value="" x="8.5" y="10" smashed="yes" rot="R90">
-<attribute name="NAME" x="7.9" y="12.75" size="0.8" layer="25"/>
+<attribute name="NAME" x="7.9" y="12.75" size="0.8" layer="25" font="vector"/>
 <attribute name="VALUE" x="9.784" y="8.9" size="0.4064" layer="27" rot="R90"/>
 </element>
 <element name="J1" library="jst-ph" package="JST-PH3" value="JST-PH3" x="12" y="4" smashed="yes" rot="R180"/>
 <element name="R2" library="adafruit" package="R1206" value="10k" x="13.5" y="10" smashed="yes" rot="R90">
-<attribute name="NAME" x="12.988" y="12.766" size="0.8" layer="25"/>
+<attribute name="NAME" x="12.988" y="12.766" size="0.8" layer="25" font="vector"/>
 <attribute name="VALUE" x="15.786" y="9.238" size="1.27" layer="27" rot="R90"/>
 </element>
 <element name="C1" library="adafruit" package="C1206" value="100n" x="6" y="10" smashed="yes" rot="R90">
-<attribute name="NAME" x="5.111" y="12.766" size="0.8" layer="25"/>
+<attribute name="NAME" x="5.111" y="12.766" size="0.8" layer="25" font="vector"/>
 <attribute name="VALUE" x="8.286" y="9.111" size="1.27" layer="27" rot="R90"/>
 </element>
+<element name="U$1" library="adafruit" package="FIDUCIAL_1MM" value="FIDUCIAL" x="6" y="5"/>
+<element name="U$2" library="adafruit" package="FIDUCIAL_1MM" value="FIDUCIAL" x="19" y="18"/>
 </elements>
 <signals>
@@
 <contactref element="Q1" pad="3"/>
 <contactref element="D1" pad="A"/>
-<polygon width="0.25" layer="1" isolate="0.5" thermals="no" rank="6">
+<polygon width="0.25" layer="1" isolate="0.4" thermals="no" rank="6">
 <vertex x="0" y="0"/>
 <vertex x="0" y="24"/>
@@
 <contactref element="R2" pad="1"/>
 <contactref element="J1" pad="3"/>
-<polygon width="0.25" layer="16" isolate="0.5" thermals="no" rank="6">
+<polygon width="0.25" layer="16" isolate="0.4" thermals="no" rank="6">
 <vertex x="0" y="0"/>
 <vertex x="0" y="24"/>
@@
 <vertex x="24" y="0"/>
 </polygon>
-<polygon width="0.25" layer="1" isolate="0.5" thermals="no" rank="5">
+<polygon width="0.25" layer="1" isolate="0.4" thermals="no" rank="5">
 <vertex x="0" y="7"/>
 <vertex x="17" y="7"/>
